Commit message: second commit

File: src/robot_model_pkg/urdf/robot.xacro (robot description, xacro)
@@ -7,8 +7,8 @@
 <xacro:property name="wheel_link_radius" value="0.06"/>
 <xacro:property name="wheel_link_length" value="0.025"/>
-<xacro:property name="wheel_link_z_location" value="-0.13"/>
+<xacro:property name="wheel_link_z_location" value="-0.07"/>
 <!--Material density-->
-<xacro:property name="body_density" value="2710.0"/>
-<xacro:property name="wheel_density" value="2710.0"/>
+<xacro:property name="body_density" value="27100.0"/><!--여기바꿈0추가-->
+<xacro:property name="wheel_density" value="27100.0"/>
 <!-- PI constant-->
 <xacro:property name="pi_const" value="3.14159265"/>
@@ -29,4 +29,7 @@
     <color rgba = "0.54 0.16 0.88 1"/>
   </material>
+  <material name="changF">
+    <color rgba = "0.7 0 0.5 1"/>
+  </material>
 <!-- This macro defines the complete inertial section of the wheel-->
 <!-- It is used later in the code -->
@@ -93,4 +96,5 @@
                         <cylinder length="${wheel_link_length}" radius="${wheel_link_radius}"/>
                 </geometry>
+                 <material name = "changF"/>
         </visual>
         <collision>
@@ -123,4 +127,5 @@
                         <cylinder length="${wheel_link_length}" radius="${wheel_link_radius}"/>
                 </geometry>
+                <material name = "changF"/>
         </visual>
         <collision>
@@ -153,4 +158,5 @@
                         <cylinder length="${wheel_link_length}" radius="${wheel_link_radius}"/>
                 </geometry>
+                <material name = "changF"/>
         </visual>
         <collision>
@@ -183,4 +189,5 @@
                         <cylinder length="${wheel_link_length}" radius="${wheel_link_radius}"/>
                 </geometry>
+                <material name = "changF"/>
         </visual>
         <collision>
@@ -193,5 +200,5 @@
 </link>
   <joint name = "head_scanner" type = "fixed">
-    <origin xyz = "0 0 0.15" rpy = "0 0 0"/>
+    <origin xyz = "0 0 0.07" rpy = "0 0 0"/>
     <parent link = "base_link"/>
     <child link = "base_scan"/>
@@ -206,7 +213,7 @@
     </visual>
     <collision>
-      <origin xyz="0 0 0.4" rpy = "0 0 1.570795"/>
+      <origin xyz="0 0 0.05" rpy = "0 0 1.570795"/>
       <geometry>
-        <cylinder length="0.09" radius="0.09"/>
+        <cylinder length="0.1" radius="0.09"/>
       </geometry>
     </collision>
