Commit message: first commit

File: src/robot_model_pkg/urdf/caps.xacro (robot description, xacro)
@@ -1,7 +1,8 @@
 <robot name="differential_drive_robot" xmlns:xacro="http://www.ros.org/wiki/xacro">
 <!-- body dimensions-->
-<xacro:property name="body_link_x_dim" value="0.397"/><!--1-->
-<xacro:property name="body_link_y_dim" value="0.320"/><!--0.6-->
-<xacro:property name="body_link_z_dim" value="0.156"/><!--0.3-->
+<!--caps -->
+<xacro:property name="body_link_x_dim" value="0.45"/><!--1-->
+<xacro:property name="body_link_y_dim" value="0.45"/><!--0.6-->
+<xacro:property name="body_link_z_dim" value="0."/><!--0.3-->
 <!-- wheel dimensions-->
 <xacro:property name="wheel_link_radius" value="0.06"/>

Commit message: first commit

File: src/robot_model_pkg/urdf/caps.xacro (robot description, xacro)
@@ -2,18 +2,20 @@
 <!-- body dimensions-->
 <!--caps -->
-<xacro:property name="body_link_x_dim" value="0.45"/><!--1-->
-<xacro:property name="body_link_y_dim" value="0.45"/><!--0.6-->
-<xacro:property name="body_link_z_dim" value="0."/><!--0.3-->
+<xacro:property name="body_link_x_dim" value="0.5"/><!--1-->
+<xacro:property name="body_link_y_dim" value="0.5"/><!--0.6-->
+<xacro:property name="body_link_z_dim" value="0.2"/><!--0.3-->
 <!-- wheel dimensions-->
-<xacro:property name="wheel_link_radius" value="0.06"/>
-<xacro:property name="wheel_link_length" value="0.025"/>
-<xacro:property name="wheel_link_z_location" value="-0.07"/>
+<xacro:property name="wheel_link_radius" value="0.17"/>
+<xacro:property name="wheel_link_length" value="0.07"/>
+<xacro:property name="wheel_link_z_location" value="-0.25"/>
+<!--caster dimensions-->
+<xacro:property name="caster_link_radius" value="0.13"/>
+<xacro:property name="caster_link_length" value="0.07"/>
 <!--Material density-->
-<xacro:property name="body_density" value="2010.0"/><!--여기바꿈0추가-->
-<xacro:property name="wheel_density" value="2010.0"/>
+<xacro:property name="wheel_density" value="201.0"/>
 <!-- PI constant-->
 <xacro:property name="pi_const" value="3.14159265"/>
 <!-- Robot body and wheel mass-->
-<xacro:property name="body_mass" value="${body_density*body_link_x_dim*body_link_y_dim*body_link_z_dim}"/>
+<xacro:property name="body_mass" value="30.0"/> <!--wheel_mass 대략1.13kg나옴-->
 <xacro:property name="wheel_mass" value="${wheel_density*pi_const*wheel_link_radius*wheel_link_radius*wheel_link_length}"/>
 <!-- Moment of inertia of the wheel-->
@@ -21,4 +23,22 @@
 <xacro:property name="I_wheel" value="${(1.0/12.0)*wheel_mass*(3.0*wheel_link_radius*wheel_link_radius+wheel_link_length*wheel_link_length)}"/>
 <!-- color -->
+<material name="metallic_grey">
+    <color rgba="0.5 0.5 0.5 1"/> <!-- 회색조의 금속을 나타내는 색상 -->
+</material>
+<material name="metallic_black">
+    <color rgba="0.2 0.2 0.2 1"/> <!--캐스터 관절 -->
+</material>
+<material name="metallic_black_bar">
+    <color rgba="0.7 0.7 0.7 1"/> <!--캐스터 관절 바 -->
+</material>
+<material name="metallic_black_bar_W">
+    <color rgba="0.9 0.9 0.9 1"/> <!--캐스터 관절 - 바퀴 연결  -->
+</material>
+<material name="mix">
+    <color rgba = "0.88 0.88 0.22 1"/>
+  </material>
+<material name="coral">
+    <color rgba = "0.99 0.55 0.3 1"/>
+  </material>
 <material name="blue">
     <color rgba = "0 0 0.8 1"/>
@@ -28,11 +48,11 @@
   </material>
   <material name="blueviolet">
-    <color rgba = "0.54 0.16 0.88 1"/>
+    <color rgba = "0.222 0.888 0.38 1"/>
   </material>
   <material name="changF">
-    <color rgba = "0.7 0 0.5 1"/>
+    <color rgba = "0.4 0.4 0.4 1"/>
   </material>
   <material name="changS">
-    <color rgba = "0.2 0.9 0.1 1"/>
+    <color rgba = "0.3 0.3 0.3 1"/>
   </material>
 <!-- This macro defines the complete inertial section of the wheel-->
@@ -63,8 +83,192 @@
         <visual>
                 <geometry>
-                        <box size="${body_link_x_dim} ${body_link_y_dim} ${body_link_z_dim}" />
-                </geometry>
-        <origin rpy="0 0 0" xyz="0 0 0" />
-        </visual>
+                        <box size="${body_link_x_dim} ${body_link_y_dim} ${body_link_z_dim-0.1}" />
+                </geometry>
+                <material name = "changF"/>
+                <origin rpy="0 0 0" xyz="0 0 0" />
+        </visual>
+        <visual>
+                <geometry>
+                        <cylinder length="0.50" radius="0.03"/>
+                </geometry>
+                  <material name="metallic_grey"/>
+                 <!--origin xyz = "0 0.30 0" rpy = "0 1.570795 0"/-->           <!--왼쪽 캐스터지지대 -->
+                 <!--origin rpy="0 1.22173 0" xyz="0 0 0" 70도 회전        각 사이드 바 5도:0.0872665        /-->
+                <origin xyz = "0 0.298 0.006" rpy = "0 1.396263 -0.0523599"/> <!--80도 회전,3도 회전-->
+        </visual>
+        <visual>
+                <geometry>
+                        <cylinder length="0.50" radius="0.03"/>
+                </geometry>
+                  <material name="metallic_grey"/>
+                 <!--origin xyz = "0 0.30 0" rpy = "0 1.570795 0"/-->
+                 <!--origin rpy="0 1.22173 0" xyz="0 0 0" 70도 회전        오른쪽 캐스터 지지대    /-->
+                <origin xyz = "0 -0.298 0.006" rpy = "0 1.396263 0.0523599"/> <!--80도 회전-->
+        </visual>
+<!--###################################left caster part ###########################################-->
+        <visual>
+                <geometry>
+                        <cylinder length="0.08" radius="0.033"/>   <!--caster 관절 부분 -->
+                </geometry>
+                  <material name="metallic_black"/>
+                 <!--origin xyz = "0 0.30 0" rpy = "0 1.570795 0"/-->
+                 <!--origin rpy="0 1.22173 0" xyz="0 0 0" 70도 회전/-->
+                <origin xyz = "-0.235 0.310 -0.035" rpy = "0 0 0"/>
+        </visual>
+        <visual>
+                <geometry>
+                        <cylinder length="0.12" radius="0.027"/>   <!--caster 관절 바 부분 -->
+                </geometry>
+                  <material name="metallic_black_bar"/>
+                 <!--origin xyz = "0 0.30 0" rpy = "0 1.570795 0"/-->
+                 <!--origin rpy="0 1.22173 0" xyz="0 0 0" 70도 회전/-->
+                <origin xyz = "-0.235 0.310 -0.035" rpy = "0 0 0"/>
+        </visual>
+        <visual>
+                <geometry>
+                        <box size= "0.05 0.1 0.01"/>        <!--caster 관절 바 - 바퀴 연결 부분 -->
+                </geometry>
+                  <material name="metallic_black_bar_W"/>
+                 <!--origin xyz = "0 0.30 0" rpy = "0 1.570795 0"/-->
+                 <!--origin rpy="0 1.22173 0" xyz="0 0 0" 70도 회전/-->
+                <origin xyz = "-0.235 0.310 -0.1" rpy = "0 0 0"/>
+        </visual>
+        <visual>
+                <geometry>
+                        <box size= "0.05 0.20 0.01"/>        <!--caster 관절 바 - 바퀴 연결 일자 겉 부분 -->
+                </geometry>
+                  <material name="metallic_black_bar_W"/>
+                 <!--origin xyz = "0 0.30 0" rpy = "0 1.570795 0"/-->
+                 <!--origin rpy="0 1.22173 0" xyz="0 0 0" 70도 회전/-->
+                <origin xyz = "-0.235 0.360 -0.20" rpy = "1.570795 0 0"/>
+        </visual>
+        <visual>
+                <geometry>
+                        <box size= "0.05 0.20 0.01"/>        <!--caster 관절 바 - 바퀴 연결 일자 속 부분 -->
+                </geometry>
+                  <material name="metallic_black_bar_W"/>
+                 <!--origin xyz = "0 0.30 0" rpy = "0 1.570795 0"/-->
+                 <!--origin rpy="0 1.22173 0" xyz="0 0 0" 70도 회전/-->
+                <origin xyz = "-0.235 0.26 -0.20" rpy = "1.570795 0 0"/>
+        </visual>
+<!--###################################Right caster part ###########################################-->
+        <visual>
+                <geometry>
+                        <cylinder length="0.08" radius="0.033"/>   <!--caster 관절 부분 -->
+                </geometry>
+                  <material name="metallic_black"/>
+                 <!--origin xyz = "0 0.30 0" rpy = "0 1.570795 0"/-->
+                 <!--origin rpy="0 1.22173 0" xyz="0 0 0" 70도 회전/-->
+                <origin xyz = "-0.235 -0.310 -0.035" rpy = "0 0 0"/>
+        </visual>
+        <visual>
+                <geometry>
+                        <cylinder length="0.12" radius="0.027"/>   <!--caster 관절 바 부분 -->
+                </geometry>
+                  <material name="metallic_black_bar"/>
+                 <!--origin xyz = "0 0.30 0" rpy = "0 1.570795 0"/-->
+                 <!--origin rpy="0 1.22173 0" xyz="0 0 0" 70도 회전/-->
+                <origin xyz = "-0.235 -0.310 -0.035" rpy = "0 0 0"/>
+        </visual>
+        <visual>
+                <geometry>
+                        <box size= "0.05 0.1 0.01"/>        <!--caster 관절 바 - 바퀴 연결 부분 -->
+                </geometry>
+                  <material name="metallic_black_bar_W"/>
+                 <!--origin xyz = "0 0.30 0" rpy = "0 1.570795 0"/-->
+                 <!--origin rpy="0 1.22173 0" xyz="0 0 0" 70도 회전/-->
+                <origin xyz = "-0.235 -0.310 -0.1" rpy = "0 0 0"/>
+        </visual>
+        <visual>
+                <geometry>
+                        <box size= "0.05 0.20 0.01"/>        <!--caster 관절 바 - 바퀴 연결 일자 밖 부분 -->
+                </geometry>
+                  <material name="metallic_black_bar_W"/>
+                 <!--origin xyz = "0 0.30 0" rpy = "0 1.570795 0"/-->
+                 <!--origin rpy="0 1.22173 0" xyz="0 0 0" 70도 회전/-->
+                <origin xyz = "-0.235 -0.360 -0.20" rpy = "1.570795 0 0"/>
+        </visual>
+        <visual>
+                <geometry>
+                        <box size= "0.05 0.20 0.01"/>        <!--caster 관절 바 - 바퀴 연결 일자 속 부분 -->
+                </geometry>
+                  <material name="metallic_black_bar_W"/>
+                 <!--origin xyz = "0 0.30 0" rpy = "0 1.570795 0"/-->
+                 <!--origin rpy="0 1.22173 0" xyz="0 0 0" 70도 회전/-->
+                <origin xyz = "-0.235 -0.26 -0.20" rpy = "1.570795 0 0"/>
+        </visual>
+<!--################################### under base ###########################################-->
+        <visual>
+                <geometry>
+                        <box size="${body_link_x_dim-0.1} ${body_link_y_dim/1.2} ${body_link_z_dim}" />
+                </geometry>
+                <material name = "metallic_black_bar_W"/>
+                <origin rpy="0 0 0" xyz="0 0 -0.1" />
+        </visual>
+        <visual>
+                <geometry>                      <!--번호판 느낌-->
+                        <box size="0.18 ${body_link_y_dim/1.2} ${body_link_z_dim/3}" />
+                </geometry>
+                <material name = "metallic_black_bar_W"/>
+                <origin rpy="0 1.919862 0" xyz="0.19 0 -0.1" />
+        </visual>
+        <visual>
+                <geometry>                      <!--번호판 느낌-->
+                        <box size="0.18 ${body_link_y_dim/1.2} ${body_link_z_dim/3}" />
+                </geometry>
+                <material name = "metallic_black_bar_W"/>
+                <origin rpy="0 -1.919862 0" xyz="-0.19 0 -0.1" />
+        </visual>
+<!--################################### drawer base ###########################################-->
+        <visual>
+                <geometry>              <!--1층 서랍-->
+                        <box size="${body_link_x_dim-0.1} ${body_link_y_dim/1.2} ${body_link_z_dim}" />
+                </geometry>
+                <material name = "metallic_black_bar_W"/>
+                <origin rpy="0 0 0" xyz="0 0 0.1" />
+        </visual>
+        <visual>
+                <geometry>              <!--1층 서랍 손잡이-->
+                        <box size="${(body_link_x_dim-0.2)/2} ${body_link_y_dim/2} ${body_link_z_dim/3.3}" />
+                </geometry>
+                <material name = "metallic_black_bar"/>
+                <origin rpy="0 0 0" xyz="0 0.095 0.1" />
+        </visual>
+        <visual>
+                <geometry>              <!--1~2층 분리대 -->
+                        <box size="${body_link_x_dim-0.099} ${body_link_y_dim/1.199} 0.01" />
+                </geometry>
+                <material name = "metallic_black"/>
+                <origin rpy="0 0 0" xyz="0 0 0.2" />
+        </visual>
+        <visual>
+                <geometry>              <!--2층 서랍-->
+                        <box size="${body_link_x_dim-0.1} ${body_link_y_dim/1.2} ${body_link_z_dim}" />
+                </geometry>
+                <material name = "metallic_black_bar_W"/>
+                <origin rpy="0 0 0" xyz="0 0 0.3" />
+        </visual>
+        <visual>
+                <geometry>              <!--2층 서랍 손잡이-->
+                        <box size="${(body_link_x_dim-0.2)/2} ${body_link_y_dim/2} ${body_link_z_dim/3.3}" />
+                </geometry>
+                <material name = "metallic_black_bar"/>
+                <origin rpy="0 0 0" xyz="0 0.095 0.28" />
+        </visual>
+        <visual>
+                <geometry>              <!--2층 UWB 센서1-->
+                        <box size="${(body_link_x_dim-0.2)/2} ${body_link_y_dim/6.5} ${body_link_z_dim/6}" />
+                </geometry>
+                <material name = "mix"/>
+                <origin rpy="1.570795 0 0" xyz="0.15 0.18 0.35" />
+        </visual>
+        <visual>
+                <geometry>              <!--2층 UWB 센서2-->
+                        <box size="${(body_link_x_dim-0.2)/2} ${body_link_y_dim/6.5} ${body_link_z_dim/6}" />
+                </geometry>
+                <material name = "mix"/>
+                <origin rpy="1.570795 0 0" xyz="0.15 -0.18 0.35" />
+        </visual>
+<!--###############################collision part #######################################-->
         <collision>
                 <geometry>
@@ -88,9 +292,9 @@
         <parent link="base_link"/>
         <child link="wheel1_link"/>
-        <origin xyz="${-body_link_x_dim/2+1.2*wheel_link_radius} ${-body_link_y_dim/2-wheel_link_length/2} ${wheel_link_z_location}"
+        <origin xyz="${-body_link_x_dim/2+3*wheel_link_radius} ${-body_link_y_dim/1.55+wheel_link_length/2} ${wheel_link_z_location}"
         rpy = "0 0 0"/>
         <axis xyz="0 1 0"/>
         <limit effort="1000" velocity="1000"/>
-        <dynamics damping="1.0" friction="1.0" />
+        <dynamics damping="0.2" friction="0.0" />
 </joint>
 <link name="wheel1_link">
@@ -100,5 +304,5 @@
                         <cylinder length="${wheel_link_length}" radius="${wheel_link_radius}"/>
                 </geometry>
-                 <material name = "changF"/>
+                 <material name = "changS"/>
         </visual>
         <collision>
@@ -119,9 +323,9 @@
         <parent link="base_link"/>
         <child link="wheel2_link"/>
-        <origin xyz="${-body_link_x_dim/2+1.2*wheel_link_radius} ${body_link_y_dim/2+wheel_link_length/2} ${wheel_link_z_location}"
+        <origin xyz="${-body_link_x_dim/2+3*wheel_link_radius} ${body_link_y_dim/2+wheel_link_length/2} ${wheel_link_z_location}"
         rpy = "0 0 0"/>
         <axis xyz="0 1 0"/>
         <limit effort="1000" velocity="1000"/>
-        <dynamics damping="1.0" friction="1.0" />
+        <dynamics damping="0.2" friction="0.0" />
 </joint>
 <link name="wheel2_link">
@@ -131,5 +335,5 @@
                         <cylinder length="${wheel_link_length}" radius="${wheel_link_radius}"/>
                 </geometry>
-                <material name = "changF"/>
+                <material name = "changS"/>
         </visual>
         <collision>
@@ -144,49 +348,92 @@
 <!-- END: BACK LEFT WHEEL OF THE ROBOT AND THE JOINT-->
 <!-- ##########################################################-->
-<!-- ##########################################################-->
-<!-- START : FRONT RIGTH WHEEL OF THE ROBOT AND THE JOINT-->
-<!-- ##########################################################-->
- <joint name = "caster_wheel_joint" type = "fixed">
-    <parent link = "base_link"/>
-    <child link = "caster_wheel"/>
-    <origin xyz="${body_link_x_dim/2-1.8*wheel_link_radius} ${-body_link_y_dim/2+0.15} ${wheel_link_z_location}"
-        rpy = "0 0 0"/>
-    <axis xyz="0 1 0"/>
-  </joint>
-   <link name="caster_wheel">
-    <visual>
-      <origin xyz="0 0 0" rpy = "1.570795 0 0"/>
-      <geometry>
-     <cylinder length="${wheel_link_length*2}" radius="${wheel_link_radius}"/>
-      </geometry>
-      <material name = "blueviolet"/>
-    </visual>
-    <collision>
-      <origin xyz="0 0 0" rpy = "1.570795 0 0"/>
-      <geometry>
- <cylinder length="${wheel_link_length*2}" radius="${wheel_link_radius}"/>
-      </geometry>
+<!--이 부분에 caster와 연결되는 joint 설정해보기 -->
+ <!--연결 바 위치 정보 origin xyz = "-0.235 -0.310 -0.035" rpy = "0 0 0"/-->
+        <!--fixed continuous-->
+<joint name="connect2caster_joint_1" type="fixed">
+        <parent link="base_link"/>
+        <child link="connect2caster_1"/>
+         <origin xyz = "-0.235 -0.310 -0.1" rpy = "0 0 0"/>
+        <axis xyz="0 0 1"/>
+        <limit effort="1000" velocity="1000"/>
+        <dynamics damping="0.2" friction="0.0" />
+</joint>
+<link name="connect2caster_1">
+        <visual>
+        <origin xyz="0 0 ${wheel_link_z_location+0.06}" rpy = "1.570795 0 0"/>
+        <geometry>
+                <cylinder length="${wheel_link_length}" radius="${caster_link_radius}"/>
+        </geometry>
+        <material name = "changS"/>
+        </visual>
+        <collision>
+         <origin xyz="0 0 ${wheel_link_z_location+0.06}" rpy = "1.570795 0 0"/>
+        <geometry>
+                <cylinder length="${wheel_link_length}" radius="${caster_link_radius}"/>
+        </geometry>
     </collision>
+    <!--xacro:inertia_wheel/-->
   </link>
+<!-- ##########################################################-->
+<!-- START : caster right & back-->
+<!--연결 바 위치 정보 origin xyz = "-0.235 -0.310 -0.035" rpy = "0 0 0"/-->
+<!-- ##########################################################-->
+<!-- START : caster left & back-->
+<joint name="connect2caster_joint_2" type="fixed">
+        <parent link="base_link"/>
+        <child link="connect2caster_2"/>
+         <origin xyz = "-0.235 +0.310 -0.1" rpy = "0 0 0"/>
+        <axis xyz="0 0 1"/>
+        <limit effort="1000" velocity="1000"/>
+        <dynamics damping="0.2" friction="0.0" />
+</joint>
+<link name="connect2caster_2">
+        <visual>
+        <origin xyz="0 0 ${wheel_link_z_location+0.06}" rpy = "1.570795 0 0"/>
+        <geometry>
+                <cylinder length="${wheel_link_length}" radius="${caster_link_radius}"/>
+        </geometry>
+        <material name = "changS"/>
+        </visual>
+        <collision>
+       <origin xyz="0 0 ${wheel_link_z_location+0.06}" rpy = "1.570795 0 0"/>
+        <geometry>
+                <cylinder length="${wheel_link_length}" radius="${caster_link_radius}"/>
+        </geometry>
+    </collision>
+    <!--xacro:inertia_wheel/-->
+  </link>
+<!-- #####################################################################-->
+<!--CASTER PART-->
+<!-- #####################################################################-->
+<!--LIDAR PART-->
   <joint name = "head_scanner" type = "fixed">
-    <origin xyz = "0 0 0.07" rpy = "0 0 0"/>
+    <origin xyz = "0 0 0.45" rpy = "0 0 0"/>
     <parent link = "base_link"/>
     <child link = "base_scan"/>
   </joint>
-   <link name="base_scan">
-    <visual>
-      <origin xyz="0 0 0.05" rpy = "0 0 1.570795"/>
-      <geometry>
-        <cylinder length="0.1" radius="0.09"/>
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